File: Water Quality Measurement/Water Quality Measurement.kicad_sch (KiCad schematic)
At the start: 14 parts, among them J1 pH Sensor, J2 OLED Screen, J3 MountingPin_IO1, J4 Conn_01x02_MountingPin, J5 MountingPin_IO46, J6 Voltage 9 ->5 regulator, Q1 2N2219, U1 LM7805_TO220

Commit message: Add files via upload
Parts:
- removed D1: 1N4007, Diode_THT:D_DO-41_SOD81_P10.16mm_Horizontal, symbol Diode:1N4007
- removed Q1: 2N2219, Package_TO_SOT_THT:TO-39-3, symbol Transistor_BJT:2N2219
- added C1: 0.1u, Capacitor_SMD:C_0805_2012Metric_Pad1.18x1.45mm_HandSolder, symbol Device:C
- added C2: 0.22u, Capacitor_SMD:C_0805_2012Metric_Pad1.18x1.45mm_HandSolder, symbol Device:C
- added J7: Conn_01x02_MountingPin, Connector_PinHeader_2.54mm:PinHeader_1x02_P2.54mm_Vertical, symbol Connector_Generic_MountingPin:Conn_01x02_MountingPin
- added J8: 9V Battery Enclosure, Connector_PinHeader_2.54mm:PinHeader_1x02_P2.54mm_Vertical, symbol Connector_Generic_MountingPin:Conn_01x02_MountingPin
- added Q1: PMV15UNEAR, Package_TO_SOT_SMD:SOT-23, symbol Device:Q_NMOS_GSD
- J6: value Voltage 9 ->5 regulator -> 9V Battery Enclosure
- R1: value R_US -> 1k
Connections:
- net GND: now also C1.2, C2.2, J8.2 (Pin_2), Q1.2 (S)
- net at R1.2: now also Q1.1 (G)
- net at J4.2 (Pin_2): now also J7.2 (Pin_2), Q1.3 (D)
- net 9V enclosure: no longer names the net of U1.1 (VI)
- net 9V enclosure: now also J4.1 (Pin_1), J6.1 (Pin_1), C2.1, J7.1 (Pin_1)
- removed net Vbatt: J4.1 (Pin_1), J6.1 (Pin_1), U1.3 (VO)
- new net: C1.1, J8.1 (Pin_1), U1.3 (VO)
Other:
- moved on the sheet: J6
